File: boards/smart_headphones/smart_headphones_rev_Nov2016.sch (EAGLE design)
At the start: 14 parts, among them U1 ATMEGA328P_PDIP

Commit message: Fixed bug (two control signals connected)
Parts:
- JP8: value (none) -> M02PTH3; device Finn-lbr-rev1:M03LONGPADS -> Finn-lbr-rev1:M02PTH3
Connections:
- removed net N$17: JP8.1, U1.PD2(INT0)
- new net PWREN: U$1.PWREN, U1.PD2(INT0)
- net N$18: now also JP8.1; no longer JP8.2
- net N$19: now also JP8.2; no longer JP8.3
- net PB6: no longer U$1.PWREN
Changed lines of the file:
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@@
 <part name="JP7" library="Finn-lbr-rev1" deviceset="M02" device="PTH3"/>
 <part name="GND" library="Finn-lbr-rev1" deviceset="GND" device=""/>
-<part name="JP8" library="Finn-lbr-rev1" deviceset="M03" device="LONGPADS"/>
 <part name="JP9" library="Finn-lbr-rev1" deviceset="M03" device="LONGPADS"/>
 <part name="JP10" library="Finn-lbr-rev1" deviceset="M02" device="PTH3"/>
@@
 <part name="SUPPLY5" library="Finn-lbr-rev1" deviceset="VCC" device=""/>
 <part name="FRAME1" library="Finn-lbr-rev1" deviceset="FRAME-LETTER" device=""/>
+<part name="JP8" library="Finn-lbr-rev1" deviceset="M02" device="PTH3"/>
 </parts>
 <sheets>
@@
 <instance part="JP7" gate="G$1" x="96.52" y="-5.08"/>
 <instance part="GND" gate="1" x="109.22" y="-12.7"/>
-<instance part="JP8" gate="G$1" x="165.1" y="58.42" rot="R180"/>
 <instance part="JP9" gate="G$1" x="223.52" y="5.08"/>
 <instance part="JP10" gate="G$1" x="259.08" y="5.08" rot="R180"/>
@@
 <instance part="FRAME1" gate="G$1" x="68.58" y="-45.72"/>
 <instance part="FRAME1" gate="G$2" x="215.9" y="-45.72"/>
+<instance part="JP8" gate="G$1" x="167.64" y="58.42" rot="R180"/>
 </instances>
 <busses>
@@
 <net name="PB6" class="0">
 <segment>
-<pinref part="U$1" gate="G$1" pin="PWREN"/>
-<wire x1="185.42" y1="116.84" x2="193.04" y2="116.84" width="0.1524" layer="91"/>
-</segment>
-<segment>
 <pinref part="U1" gate="G$1" pin="PB6(XTAL1/TOSC1)"/>
 <wire x1="93.98" y1="66.04" x2="81.28" y2="66.04" width="0.1524" layer="91"/>
@@
 </segment>
 </net>
-<net name="N$17" class="0">
-<segment>
-<pinref part="U1" gate="G$1" pin="PD2(INT0)"/>
-<pinref part="JP8" gate="G$1" pin="1"/>
-<wire x1="142.24" y1="63.5" x2="157.48" y2="63.5" width="0.1524" layer="91"/>
-<wire x1="157.48" y1="63.5" x2="157.48" y2="60.96" width="0.1524" layer="91"/>
-</segment>
-</net>
 <net name="N$18" class="0">
 <segment>
@@
 <wire x1="142.24" y1="60.96" x2="154.94" y2="60.96" width="0.1524" layer="91"/>
 <wire x1="154.94" y1="60.96" x2="154.94" y2="58.42" width="0.1524" layer="91"/>
-<wire x1="154.94" y1="58.42" x2="157.48" y2="58.42" width="0.1524" layer="91"/>
-<pinref part="JP8" gate="G$1" pin="2"/>
-<wire x1="160.02" y1="58.42" x2="157.48" y2="58.42" width="0.1524" layer="91"/>
+<wire x1="160.02" y1="58.42" x2="154.94" y2="58.42" width="0.1524" layer="91"/>
+<pinref part="JP8" gate="G$1" pin="1"/>
 </segment>
 </net>
@@
 <wire x1="142.24" y1="58.42" x2="152.4" y2="58.42" width="0.1524" layer="91"/>
 <wire x1="152.4" y1="58.42" x2="152.4" y2="55.88" width="0.1524" layer="91"/>
-<pinref part="JP8" gate="G$1" pin="3"/>
-<wire x1="152.4" y1="55.88" x2="157.48" y2="55.88" width="0.1524" layer="91"/>
+<wire x1="152.4" y1="55.88" x2="160.02" y2="55.88" width="0.1524" layer="91"/>
+<pinref part="JP8" gate="G$1" pin="2"/>
 </segment>
 </net>
@@
 </segment>
 </net>
+<net name="PWREN" class="0">
+<segment>
+<pinref part="U$1" gate="G$1" pin="PWREN"/>
+<wire x1="193.04" y1="116.84" x2="185.42" y2="116.84" width="0.1524" layer="91"/>
+</segment>
+<segment>
+<pinref part="U1" gate="G$1" pin="PD2(INT0)"/>
+<wire x1="142.24" y1="63.5" x2="157.48" y2="63.5" width="0.1524" layer="91"/>
+<wire x1="157.48" y1="63.5" x2="157.48" y2="60.96" width="0.1524" layer="91"/>
+</segment>
+</net>
